Commit message: 0.3ver

File: sim/sim_description/urdf/xacro/main.xacro (robot description, xacro)
@@ -226,5 +226,5 @@
             <updateRate>50.0</updateRate>
             <bodyName>ee_link</bodyName>
-            <topicName>wrist_pose_ground_truth</topicName>
+            <topicName>ee_pose_ground_truth</topicName>
             <gaussianNoise>0.0</gaussianNoise>
             <frameName>world</frameName>

File: sim/sim_description/urdf/xacro/ur5e.urdf.xacro (robot description, xacro)
@@ -10,10 +10,12 @@
       <mass value="${mass}" />
       <xacro:insert_block name="origin" />
-      <inertia ixx="${0.0833333 * mass * (3 * radius * radius + length * length)}" ixy="0.0" ixz="0.0"
+      <inertia ixx="${0.0833333 * mass * (3 * radius * radius + length * length)}" ixy="0.0"
+        ixz="0.0"
         iyy="${0.0833333 * mass * (3 * radius * radius + length * length)}" iyz="0.0"
         izz="${0.5 * mass * radius * radius}" />
     </inertial>
   </xacro:macro>
-  <xacro:macro name="ur5e_robot" params="prefix joint_limited
+  <xacro:macro name="ur5e_robot"
+    params="prefix joint_limited
     shoulder_pan_lower_limit:=${-2.0 * pi}    shoulder_pan_upper_limit:=${2.0 * pi}
     shoulder_lift_lower_limit:=${--2.0 * pi}    shoulder_lift_upper_limit:=${2.0 * pi}
@@ -49,5 +51,6 @@
       joint_direction = [-1, -1, 1, 1, 1, 1]
       mass = [3.7000, 8.3930, 2.2750, 1.2190, 1.2190, 0.1879]
-      center_of_mass = [ [0, -0.02561, 0.00193], [0.2125, 0, 0.11336], [0.11993, 0.0, 0.0265], [0, -0.0018, 0.01634], [0, 0.0018,0.01634], [0, 0, -0.001159] ]
+      center_of_mass = [ [0, -0.02561, 0.00193], [0.2125, 0, 0.11336], [0.11993, 0.0, 0.0265], [0,
+    -0.0018, 0.01634], [0, 0.0018,0.01634], [0, 0, -0.001159] ]
     -->
     <xacro:property name="d1" value="0.163" />
@@ -67,12 +70,22 @@
     <xacro:property name="wrist_2_length" value="${d5}" />
     <xacro:property name="wrist_3_length" value="${d6}" />
-    <!--property name="shoulder_height" value="0.089159" /-->
-    <!--property name="shoulder_offset" value="0.13585" /-->  <!-- shoulder_offset - elbow_offset + wrist_1_length = 0.10915 -->
-    <!--property name="upper_arm_length" value="0.42500" /-->
-    <!--property name="elbow_offset" value="0.1197" /-->       <!-- CAD measured -->
-    <!--property name="forearm_length" value="0.39225" /-->
-    <!--property name="wrist_1_length" value="0.093" /-->     <!-- CAD measured -->
-    <!--property name="wrist_2_length" value="0.09465" /-->   <!-- In CAD this distance is 0.930, but in the spec it is 0.09465 -->
-    <!--property name="wrist_3_length" value="0.0823" /-->
+    <!--property
+    name="shoulder_height" value="0.089159" /-->
+    <!--property
+    name="shoulder_offset" value="0.13585" /-->  <!-- shoulder_offset - elbow_offset +
+    wrist_1_length = 0.10915 -->
+    <!--property
+    name="upper_arm_length" value="0.42500" /-->
+    <!--property
+    name="elbow_offset" value="0.1197" /-->       <!-- CAD measured -->
+    <!--property
+    name="forearm_length" value="0.39225" /-->
+    <!--property
+    name="wrist_1_length" value="0.093" /-->     <!-- CAD measured -->
+    <!--property
+    name="wrist_2_length" value="0.09465" /-->   <!-- In CAD this distance is 0.930, but in
+    the spec it is 0.09465 -->
+    <!--property
+    name="wrist_3_length" value="0.0823" /-->
     <xacro:property name="shoulder_radius" value="0.060" />   <!-- manually measured -->
     <xacro:property name="upper_arm_radius" value="0.054" />  <!-- manually measured -->
@@ -80,5 +93,5 @@
     <xacro:property name="forearm_radius" value="0.040" />    <!-- manually measured -->
     <xacro:property name="wrist_radius" value="0.045" />      <!-- manually measured -->
-    <link name="${prefix}base_link" >
+    <link name="${prefix}base_link">
       <visual>
         <geometry>
@@ -86,5 +99,5 @@
         </geometry>
         <material name="LightGrey">
-          <color rgba="0.7 0.7 0.7 1.0"/>
+          <color rgba="0.7 0.7 0.7 1.0" />
         </material>
       </visual>
@@ -100,20 +113,25 @@
     <joint name="${prefix}shoulder_pan_joint" type="revolute">
       <parent link="${prefix}base_link" />
-      <child link = "${prefix}shoulder_link" />
+      <child link="${prefix}shoulder_link" />
       <origin xyz="0.0 0.0 ${shoulder_height}" rpy="0.0 0.0 0.0" />
       <axis xyz="0 0 1" />
       <xacro:unless value="${joint_limited}">
-        <limit lower="${-2.0 * pi}" upper="${2.0 * pi}" effort="150.0" velocity="3.14"/>
-        <xacro:if value="${safety_limits}">
-          <safety_controller soft_lower_limit="${-2.0 * pi + safety_pos_margin}" soft_upper_limit="${2.0 * pi - safety_pos_margin}" k_position="${safety_k_position}" k_velocity="0.0"/>
-        </xacro:if>
-      </xacro:unless>
-      <xacro:if value="${joint_limited}">
-        <limit lower="${shoulder_pan_lower_limit}" upper="${shoulder_pan_upper_limit}" effort="150.0" velocity="3.14"/>
-        <xacro:if value="${safety_limits}">
-          <safety_controller soft_lower_limit="${shoulder_pan_lower_limit + safety_pos_margin}" soft_upper_limit="${shoulder_pan_upper_limit - safety_pos_margin}" k_position="${safety_k_position}" k_velocity="0.0"/>
-        </xacro:if>
-      </xacro:if>
-      <dynamics damping="0.0" friction="0.0"/>
+        <limit lower="${-2.0 * pi}" upper="${2.0 * pi}" effort="150.0" velocity="3.14" />
+        <xacro:if value="${safety_limits}">
+          <safety_controller soft_lower_limit="${-2.0 * pi + safety_pos_margin}"
+            soft_upper_limit="${2.0 * pi - safety_pos_margin}" k_position="${safety_k_position}"
+            k_velocity="0.0" />
+        </xacro:if>
+      </xacro:unless>
+      <xacro:if value="${joint_limited}">
+        <limit lower="${shoulder_pan_lower_limit}" upper="${shoulder_pan_upper_limit}"
+          effort="150.0" velocity="3.14" />
+        <xacro:if value="${safety_limits}">
+          <safety_controller soft_lower_limit="${shoulder_pan_lower_limit + safety_pos_margin}"
+            soft_upper_limit="${shoulder_pan_upper_limit - safety_pos_margin}"
+            k_position="${safety_k_position}" k_velocity="0.0" />
+        </xacro:if>
+      </xacro:if>
+      <dynamics damping="0.0" friction="0.0" />
     </joint>
     <link name="${prefix}shoulder_link">
@@ -123,5 +141,5 @@
         </geometry>
         <material name="LightGrey">
-          <color rgba="0.7 0.7 0.7 1.0"/>
+          <color rgba="0.7 0.7 0.7 1.0" />
         </material>
       </visual>
@@ -137,20 +155,25 @@
     <joint name="${prefix}shoulder_lift_joint" type="revolute">
       <parent link="${prefix}shoulder_link" />
-      <child link = "${prefix}upper_arm_link" />
+      <child link="${prefix}upper_arm_link" />
       <origin xyz="0.0 ${shoulder_offset} 0.0" rpy="0.0 ${pi / 2.0} 0.0" />
       <axis xyz="0 1 0" />
       <xacro:unless value="${joint_limited}">
-        <limit lower="${-2.0 * pi}" upper="${2.0 * pi}" effort="150.0" velocity="3.14"/>
-        <xacro:if value="${safety_limits}">
-          <safety_controller soft_lower_limit="${-2.0 * pi + safety_pos_margin}" soft_upper_limit="${2.0 * pi - safety_pos_margin}" k_position="${safety_k_position}" k_velocity="0.0"/>
-        </xacro:if>
-      </xacro:unless>
-      <xacro:if value="${joint_limited}">
-        <limit lower="${shoulder_lift_lower_limit}" upper="${shoulder_lift_upper_limit}" effort="150.0" velocity="3.14"/>
-        <xacro:if value="${safety_limits}">
-          <safety_controller soft_lower_limit="${shoulder_lift_lower_limit + safety_pos_margin}" soft_upper_limit="${shoulder_lift_upper_limit - safety_pos_margin}" k_position="${safety_k_position}" k_velocity="0.0"/>
-        </xacro:if>
-      </xacro:if>
-      <dynamics damping="0.0" friction="0.0"/>
+        <limit lower="${-2.0 * pi}" upper="${2.0 * pi}" effort="150.0" velocity="3.14" />
+        <xacro:if value="${safety_limits}">
+          <safety_controller soft_lower_limit="${-2.0 * pi + safety_pos_margin}"
+            soft_upper_limit="${2.0 * pi - safety_pos_margin}" k_position="${safety_k_position}"
+            k_velocity="0.0" />
+        </xacro:if>
+      </xacro:unless>
+      <xacro:if value="${joint_limited}">
+        <limit lower="${shoulder_lift_lower_limit}" upper="${shoulder_lift_upper_limit}"
+          effort="150.0" velocity="3.14" />
+        <xacro:if value="${safety_limits}">
+          <safety_controller soft_lower_limit="${shoulder_lift_lower_limit + safety_pos_margin}"
+            soft_upper_limit="${shoulder_lift_upper_limit - safety_pos_margin}"
+            k_position="${safety_k_position}" k_velocity="0.0" />
+        </xacro:if>
+      </xacro:if>
+      <dynamics damping="0.0" friction="0.0" />
     </joint>
     <link name="${prefix}upper_arm_link">
@@ -160,5 +183,5 @@
         </geometry>
         <material name="LightGrey">
-          <color rgba="0.7 0.7 0.7 1.0"/>
+          <color rgba="0.7 0.7 0.7 1.0" />
         </material>
       </visual>
@@ -174,20 +197,25 @@
     <joint name="${prefix}elbow_joint" type="revolute">
       <parent link="${prefix}upper_arm_link" />
-      <child link = "${prefix}forearm_link" />
+      <child link="${prefix}forearm_link" />
       <origin xyz="0.0 ${elbow_offset} ${upper_arm_length}" rpy="0.0 0.0 0.0" />
       <axis xyz="0 1 0" />
       <xacro:unless value="${joint_limited}">
-        <limit lower="${-pi}" upper="${pi}" effort="150.0" velocity="3.14"/>
-        <xacro:if value="${safety_limits}">
-          <safety_controller soft_lower_limit="${-2.0 * pi + safety_pos_margin}" soft_upper_limit="${2.0 * pi - safety_pos_margin}" k_position="${safety_k_position}" k_velocity="0.0"/>
-        </xacro:if>
-      </xacro:unless>
-      <xacro:if value="${joint_limited}">
-        <limit lower="${elbow_joint_lower_limit}" upper="${elbow_joint_upper_limit}" effort="150.0" velocity="3.14"/>
-        <xacro:if value="${safety_limits}">
-          <safety_controller soft_lower_limit="${elbow_joint_lower_limit + safety_pos_margin}" soft_upper_limit="${elbow_joint_upper_limit - safety_pos_margin}" k_position="${safety_k_position}" k_velocity="0.0"/>
-        </xacro:if>
-      </xacro:if>
-      <dynamics damping="0.0" friction="0.0"/>
+        <limit lower="${-pi}" upper="${pi}" effort="150.0" velocity="3.14" />
+        <xacro:if value="${safety_limits}">
+          <safety_controller soft_lower_limit="${-2.0 * pi + safety_pos_margin}"
+            soft_upper_limit="${2.0 * pi - safety_pos_margin}" k_position="${safety_k_position}"
+            k_velocity="0.0" />
+        </xacro:if>
+      </xacro:unless>
+      <xacro:if value="${joint_limited}">
+        <limit lower="${elbow_joint_lower_limit}" upper="${elbow_joint_upper_limit}" effort="150.0"
+          velocity="3.14" />
+        <xacro:if value="${safety_limits}">
+          <safety_controller soft_lower_limit="${elbow_joint_lower_limit + safety_pos_margin}"
+            soft_upper_limit="${elbow_joint_upper_limit - safety_pos_margin}"
+            k_position="${safety_k_position}" k_velocity="0.0" />
+        </xacro:if>
+      </xacro:if>
+      <dynamics damping="0.0" friction="0.0" />
     </joint>
     <link name="${prefix}forearm_link">
@@ -197,5 +225,5 @@
         </geometry>
         <material name="LightGrey">
-          <color rgba="0.7 0.7 0.7 1.0"/>
+          <color rgba="0.7 0.7 0.7 1.0" />
         </material>
       </visual>
@@ -211,20 +239,25 @@
     <joint name="${prefix}wrist_1_joint" type="revolute">
       <parent link="${prefix}forearm_link" />
-      <child link = "${prefix}wrist_1_link" />
+      <child link="${prefix}wrist_1_link" />
       <origin xyz="0.0 0.0 ${forearm_length}" rpy="0.0 ${pi / 2.0} 0.0" />
       <axis xyz="0 1 0" />
       <xacro:unless value="${joint_limited}">
-        <limit lower="${-2.0 * pi}" upper="${2.0 * pi}" effort="28.0" velocity="6.28"/>
-        <xacro:if value="${safety_limits}">
-          <safety_controller soft_lower_limit="${-2.0 * pi + safety_pos_margin}" soft_upper_limit="${2.0 * pi - safety_pos_margin}" k_position="${safety_k_position}" k_velocity="0.0"/>
-        </xacro:if>
-      </xacro:unless>
-      <xacro:if value="${joint_limited}">
-        <limit lower="${wrist_1_lower_limit}" upper="${wrist_1_upper_limit}" effort="28.0" velocity="6.28"/>
-        <xacro:if value="${safety_limits}">
-          <safety_controller soft_lower_limit="${wrist_1_lower_limit + safety_pos_margin}" soft_upper_limit="${wrist_1_upper_limit - safety_pos_margin}" k_position="${safety_k_position}" k_velocity="0.0"/>
-        </xacro:if>
-      </xacro:if>
-      <dynamics damping="0.0" friction="0.0"/>
+        <limit lower="${-2.0 * pi}" upper="${2.0 * pi}" effort="28.0" velocity="6.28" />
+        <xacro:if value="${safety_limits}">
+          <safety_controller soft_lower_limit="${-2.0 * pi + safety_pos_margin}"
+            soft_upper_limit="${2.0 * pi - safety_pos_margin}" k_position="${safety_k_position}"
+            k_velocity="0.0" />
+        </xacro:if>
+      </xacro:unless>
+      <xacro:if value="${joint_limited}">
+        <limit lower="${wrist_1_lower_limit}" upper="${wrist_1_upper_limit}" effort="28.0"
+          velocity="6.28" />
+        <xacro:if value="${safety_limits}">
+          <safety_controller soft_lower_limit="${wrist_1_lower_limit + safety_pos_margin}"
+            soft_upper_limit="${wrist_1_upper_limit - safety_pos_margin}"
+            k_position="${safety_k_position}" k_velocity="0.0" />
+        </xacro:if>
+      </xacro:if>
+      <dynamics damping="0.0" friction="0.0" />
     </joint>
     <link name="${prefix}wrist_1_link">
@@ -234,5 +267,5 @@
         </geometry>
         <material name="LightGrey">
-          <color rgba="0.7 0.7 0.7 1.0"/>
+          <color rgba="0.7 0.7 0.7 1.0" />
         </material>
       </visual>
@@ -248,20 +281,25 @@
     <joint name="${prefix}wrist_2_joint" type="revolute">
       <parent link="${prefix}wrist_1_link" />
-      <child link = "${prefix}wrist_2_link" />
+      <child link="${prefix}wrist_2_link" />
       <origin xyz="0.0 ${wrist_1_length} 0.0" rpy="0.0 0.0 0.0" />
       <axis xyz="0 0 1" />
       <xacro:unless value="${joint_limited}">
-        <limit lower="${-2.0 * pi}" upper="${2.0 * pi}" effort="28.0" velocity="6.28"/>
-        <xacro:if value="${safety_limits}">
-          <safety_controller soft_lower_limit="${-2.0 * pi + safety_pos_margin}" soft_upper_limit="${2.0 * pi - safety_pos_margin}" k_position="${safety_k_position}" k_velocity="0.0"/>
-        </xacro:if>
-      </xacro:unless>
-      <xacro:if value="${joint_limited}">
-        <limit lower="${wrist_2_lower_limit}" upper="${wrist_2_upper_limit}" effort="28.0" velocity="6.28"/>
-        <xacro:if value="${safety_limits}">
-          <safety_controller soft_lower_limit="${wrist_2_lower_limit + safety_pos_margin}" soft_upper_limit="${wrist_2_upper_limit - safety_pos_margin}" k_position="${safety_k_position}" k_velocity="0.0"/>
-        </xacro:if>
-      </xacro:if>
-      <dynamics damping="0.0" friction="0.0"/>
+        <limit lower="${-2.0 * pi}" upper="${2.0 * pi}" effort="28.0" velocity="6.28" />
+        <xacro:if value="${safety_limits}">
+          <safety_controller soft_lower_limit="${-2.0 * pi + safety_pos_margin}"
+            soft_upper_limit="${2.0 * pi - safety_pos_margin}" k_position="${safety_k_position}"
+            k_velocity="0.0" />
+        </xacro:if>
+      </xacro:unless>
+      <xacro:if value="${joint_limited}">
+        <limit lower="${wrist_2_lower_limit}" upper="${wrist_2_upper_limit}" effort="28.0"
+          velocity="6.28" />
+        <xacro:if value="${safety_limits}">
+          <safety_controller soft_lower_limit="${wrist_2_lower_limit + safety_pos_margin}"
+            soft_upper_limit="${wrist_2_upper_limit - safety_pos_margin}"
+            k_position="${safety_k_position}" k_velocity="0.0" />
+        </xacro:if>
+      </xacro:if>
+      <dynamics damping="0.0" friction="0.0" />
     </joint>
     <link name="${prefix}wrist_2_link">
@@ -271,5 +309,5 @@
         </geometry>
         <material name="LightGrey">
-          <color rgba="0.7 0.7 0.7 1.0"/>
+          <color rgba="0.7 0.7 0.7 1.0" />
         </material>
       </visual>
@@ -285,20 +323,25 @@
     <joint name="${prefix}wrist_3_joint" type="revolute">
       <parent link="${prefix}wrist_2_link" />
-      <child link = "${prefix}wrist_3_link" />
+      <child link="${prefix}wrist_3_link" />
       <origin xyz="0.0 0.0 ${wrist_2_length}" rpy="0.0 0.0 0.0" />
       <axis xyz="0 1 0" />
       <xacro:unless value="${joint_limited}">
-        <limit lower="${-2.0 * pi}" upper="${2.0 * pi}" effort="28.0" velocity="6.28"/>
-        <xacro:if value="${safety_limits}">
-          <safety_controller soft_lower_limit="${-2.0 * pi + safety_pos_margin}" soft_upper_limit="${2.0 * pi - safety_pos_margin}" k_position="${safety_k_position}" k_velocity="0.0"/>
-        </xacro:if>
-      </xacro:unless>
-      <xacro:if value="${joint_limited}">
-        <limit lower="${wrist_3_lower_limit}" upper="${wrist_3_upper_limit}" effort="28.0" velocity="6.28"/>
-        <xacro:if value="${safety_limits}">
-          <safety_controller soft_lower_limit="${wrist_3_lower_limit + safety_pos_margin}" soft_upper_limit="${wrist_3_upper_limit - safety_pos_margin}" k_position="${safety_k_position}" k_velocity="0.0"/>
-        </xacro:if>
-      </xacro:if>
-      <dynamics damping="0.0" friction="0.0"/>
+        <limit lower="${-2.0 * pi}" upper="${2.0 * pi}" effort="28.0" velocity="6.28" />
+        <xacro:if value="${safety_limits}">
+          <safety_controller soft_lower_limit="${-2.0 * pi + safety_pos_margin}"
+            soft_upper_limit="${2.0 * pi - safety_pos_margin}" k_position="${safety_k_position}"
+            k_velocity="0.0" />
+        </xacro:if>
+      </xacro:unless>
+      <xacro:if value="${joint_limited}">
+        <limit lower="${wrist_3_lower_limit}" upper="${wrist_3_upper_limit}" effort="28.0"
+          velocity="6.28" />
+        <xacro:if value="${safety_limits}">
+          <safety_controller soft_lower_limit="${wrist_3_lower_limit + safety_pos_margin}"
+            soft_upper_limit="${wrist_3_upper_limit - safety_pos_margin}"
+            k_position="${safety_k_position}" k_velocity="0.0" />
+        </xacro:if>
+      </xacro:if>
+      <dynamics damping="0.0" friction="0.0" />
     </joint>
     <link name="${prefix}wrist_3_link">
@@ -308,5 +351,5 @@
         </geometry>
         <material name="LightGrey">
-          <color rgba="0.7 0.7 0.7 1.0"/>
+          <color rgba="0.7 0.7 0.7 1.0" />
         </material>
       </visual>
@@ -322,5 +365,5 @@
     <joint name="${prefix}ee_fixed_joint" type="fixed">
       <parent link="${prefix}wrist_3_link" />
-      <child link = "${prefix}ee_link" />
+      <child link="${prefix}ee_link" />
       <origin xyz="0.0 ${wrist_3_length} 0.0" rpy="0.0 0.0 ${pi/2.0}" />
     </joint>
@@ -328,35 +371,35 @@
       <collision>
         <geometry>
-          <box size="0.01 0.01 0.01"/>
-        </geometry>
-        <origin rpy="0 0 0" xyz="-0.01 0 0"/>
+          <box size="0.01 0.01 0.01" />
+        </geometry>
+        <origin rpy="0 0 0" xyz="-0.01 0 0" />
       </collision>
     </link>
     <link name="robotiq_coupler">
-        <visual>
-        <geometry>
-            <mesh filename="package://sim_description/meshes/robotiq/robotiq_85_coupler.stl" />
-        </geometry>
-        <material name="flat_black"/>
-        </visual>
-        <collision>
-        <geometry>
-            <mesh filename="package://sim_description/meshes/robotiq/robotiq_85_coupler.stl" />
-        </geometry>
-        </collision>
-        <inertial>
-            <origin xyz="2.073e-05   1.45286e-03  -1.1049e-03" rpy="0 0 0" />
-            <mass value="0.168" />
-            <inertia ixx="6.69695624e-05" ixy="5.21511788e-09" ixz="-2.74383009e-08"
-                     iyy="7.85088161e-05" iyz="5.41105193e-07" izz="1.41819717e-04"/>
-        </inertial>
+      <visual>
+        <geometry>
+          <mesh filename="package://sim_description/meshes/robotiq/robotiq_85_coupler.stl" />
+        </geometry>
+        <material name="flat_black" />
+      </visual>
+      <collision>
+        <geometry>
+          <mesh filename="package://sim_description/meshes/robotiq/robotiq_85_coupler.stl" />
+        </geometry>
+      </collision>
+      <inertial>
+        <origin xyz="2.073e-05   1.45286e-03  -1.1049e-03" rpy="0 0 0" />
+        <mass value="0.168" />
+        <inertia ixx="6.69695624e-05" ixy="5.21511788e-09" ixz="-2.74383009e-08"
+          iyy="7.85088161e-05" iyz="5.41105193e-07" izz="1.41819717e-04" />
+      </inertial>
     </link>
     <joint name="robotiq_coupler_joint" type="fixed">
-        <origin xyz="0  0  0" rpy="1.5708 0 1.5708" />
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
Commit message: brick

File: sim/sim_description/urdf/xacro/main.xacro (robot description, xacro)
@@ -24,5 +24,5 @@
             <origin xyz="0 0 0" rpy="0 0 0" />
             <geometry>
-                <box size="1.0 1.0 0.1" />
+                <box size="0.7 0.7 0.1" />
             </geometry>
         </visual>
